File: KiCad/FatGary-devboard.sch (KiCad schematic (older format))
At the start: 9 parts, among them J1 USB_B_Micro, J2 Conn_02x01, J3 Conn_01x01, U1 PLCC-84-Plug, U2 Fat_Gary_SMD_socket, U3 Fat_Gary_TH_socket

Commit message: Change to footprint with longer pads for the PLCC-84 smd plug
Parts:
- U1: footprint FatGary-devboard:PLCC-84_Plug_P1.27mm_mirrored -> FatGary-devboard:PLCC-84_Plug_P1.27mm_mirrored_extended_pads
Changed lines of the file:
@@
 F 0 "U1" H 2050 3350 50  0000 C CNN
 F 1 "PLCC-84-Plug" H 2050 3450 50  0000 C CNN
-F 2 "FatGary-devboard:PLCC-84_Plug_P1.27mm_mirrored" H 2450 5950 50  0001 L CIN
+F 2 "FatGary-devboard:PLCC-84_Plug_P1.27mm_mirrored_extended_pads" H 2450 5950 50  0001 L CIN
 F 3 "" H 2050 3650 50  0001 C CNN
 	1    2050 3450
